File: pimicro2040.kicad_sch (KiCad schematic)
At the start: 37 parts, among them J1 Left, J2 Right, J3 Bottom, SW1 RESET, SW2 USB BOOT, U1 RP2040, U2 W25Q32JWUUIQ, U3 TLV73333PDBVR, Y1 X322512MSB4SI

Commit message: Bulk update to rev2
* Rename to PiMicro2040
* Fix critical error cause by 2-pin crystal symbol vs. 4-pin footprint
* Use Elite-C/nice\!nano-like outline
* Use mid-mounted USB-C connector
* Use a "standard" Sparkfun Pro Micro-compatible pinout
* Add 350 mA resettable fuse
* Add VBUS sensing
* Break-out USB data lines
Parts:
- added C9: 1u, Capacitor_SMD:C_0402_1005Metric, symbol Device:C
- added D1: 1N5819WS, Diode_SMD:D_SOD-323F, symbol Device:D_Schottky_Small
- added F1: 350 mA, Resistor_SMD:R_0805_2012Metric, symbol Device:Polyfuse_Small
- added R11: 5.1k, Resistor_SMD:R_0402_1005Metric, symbol Device:R
- added R12: 10k, Resistor_SMD:R_0402_1005Metric, symbol Device:R
- J1: footprint 42keebs:PinHeader_1x12_P2.54mm_Vertical_Plain -> 42keebs:PinHeader_1x13_P2.54mm_Vertical_ProMicro-Left; symbol Connector_Generic:Conn_01x12 -> Connector_Generic:Conn_01x13
- J2: footprint 42keebs:PinHeader_1x12_P2.54mm_Vertical_Plain -> 42keebs:PinHeader_1x13_P2.54mm_Vertical_ProMicro-Right; symbol Connector_Generic:Conn_01x12 -> Connector_Generic:Conn_01x13
- LOGO1, LOGO2: now left out of the parts list
- SW2: value USB BOOT -> BOOT
- USB1: value HRO-TYPE-C-31-M-12 -> HRO-TYPE-C-31-M-13; footprint Type-C:HRO-TYPE-C-31-M-12 -> 42keebs:Molex-216990_GCT-USB45xx_HRO-TYPE-C-31-M-13x-PiMicro
- Y1: symbol Device:Crystal -> Device:Crystal_GND24
- renumbered C8 to C7, C9 to C8
Connections:
- net +3V3: now also J2.5 (Pin_5), C9.1; no longer J2.4 (Pin_4)
- net D0/TX: now also J1.2 (Pin_2); no longer J1.1 (Pin_1)
- net D12: now also J3.1 (Pin_1); no longer J3.3 (Pin_3)
- net D13: now also J3.2 (Pin_2); no longer J3.4 (Pin_4)
- net D14: now also J3.3 (Pin_3); no longer J3.5 (Pin_5)
- net D1/RX: now also J1.3 (Pin_3); no longer J1.2 (Pin_2)
- net D20: now also J2.11 (Pin_11); no longer J2.10 (Pin_10)
- net D21: now also J2.13 (Pin_13); no longer J2.9 (Pin_9)
- net D26/A0: now also J2.9 (Pin_9); no longer J2.8 (Pin_8)
- net D27/A1: now also J2.8 (Pin_8); no longer J2.7 (Pin_7)
- net D28/A2: now also J2.7 (Pin_7); no longer J2.6 (Pin_6)
- net D29/A3: now also J2.6 (Pin_6); no longer J2.5 (Pin_5)
- net D2/SDA: now also J1.6 (Pin_6); no longer J1.5 (Pin_5)
- net D3/SCL: now also J1.7 (Pin_7); no longer J1.6 (Pin_6)
- net D4: now also J1.8 (Pin_8); no longer J1.7 (Pin_7)
- net D5: now also J1.9 (Pin_9); no longer J1.8 (Pin_8)
- net D6: now also J1.10 (Pin_10); no longer J1.9 (Pin_9)
- net D7: now also J1.11 (Pin_11); no longer J1.10 (Pin_10)
- net D8: now also J1.12 (Pin_12); no longer J1.11 (Pin_11)
- net D9: now also J1.13 (Pin_13); no longer J1.12 (Pin_12)
- net GND: now also J1.5 (Pin_5), J2.3 (Pin_3), Y1.2, Y1.4, C9.2, R12.1; no longer J1.3 (Pin_3), J2.2 (Pin_2)
- net VBUS: now also F1.1, R11.2; no longer C1.1, J2.1 (Pin_1), U3.1 (IN), U3.3 (EN)
- net ~{RESET}: now also J2.4 (Pin_4); no longer J2.3 (Pin_3)
- net at C4.1, R5.2: now also Y1.3; no longer Y1.2
- net D-: now reaches R3.1, USB1.5 (DN2), USB1.7 (DN1)
- net D-: now also J2.1 (Pin_1)
- net D+: now reaches R4.1, USB1.6 (DP1), USB1.8 (DP2)
- net D+: now also J1.1 (Pin_1)
- net D15: now reaches U1.18 (GPIO15)
- net D15: now also J3.4 (Pin_4)
- net D16: now reaches U1.27 (GPIO16)
- net D16: now also J3.5 (Pin_5)
- net D22: now reaches U1.34 (GPIO22)
- net D22: now also J2.10 (Pin_10)
- net D23: now reaches U1.35 (GPIO23)
- net D23: now also J2.12 (Pin_12)
- net D10: no longer names the net of U1.13 (GPIO10)
- net D10: no longer J3.1 (Pin_1)
- net D11: no longer names the net of U1.14 (GPIO11)
- net D11: no longer J3.2 (Pin_2)
- net D18: no longer names the net of U1.29 (GPIO18)
- net D18: no longer J2.12 (Pin_12)
- net D19: no longer names the net of U1.30 (GPIO19)
- net D19: now also R11.1, R12.2; no longer J2.11 (Pin_11)
- new net: D1.2 (A), F1.2
- new net RAW: C1.1, D1.1 (K), J2.2 (Pin_2), U3.1 (IN), U3.3 (EN)
- no-connect marks 11 -> 10
Other:
- moved on the sheet: C10, C11, C12, C13, C14, C15, C16, C5, C6, R10, R3, R4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

Commit message: Rev3 update
* Use HRO-TYPE-C-31-M-14
* Use 500 mA fuse instead of 350 mA one
* Improve layout (move USB termination resistors closer to MCU)
Parts:
- F1: value 350 mA -> 500 mA
- USB1: footprint 42keebs:Molex-216990_GCT-USB45xx_HRO-TYPE-C-31-M-13x-PiMicro -> 42keebs:TYPE-C-31-M-14-PiMicro
Changed lines of the file:
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@@
       (effects (font (size 1.27 1.27)) (justify left))
     )
-    (property "Value" "350 mA" (id 1) (at 30.48 100.9649 0)
+    (property "Value" "500 mA" (id 1) (at 30.48 100.9649 0)
       (effects (font (size 1.27 1.27)) (justify left))
     )
@@
       (effects (font (size 1.524 1.524)))
     )
-    (property "Footprint" "42keebs:Molex-216990_GCT-USB45xx_HRO-TYPE-C-31-M-13x-PiMicro" (id 2) (at 34.925 52.705 0)
+    (property "Footprint" "42keebs:TYPE-C-31-M-14-PiMicro" (id 2) (at 34.925 52.705 0)
       (effects (font (size 1.524 1.524)) hide)
     )
@@
     )
     (path "/1cbc711f-80b0-45aa-94e6-0b22f9359dc1"
-      (reference "F1") (unit 1) (value "350 mA") (footprint "Resistor_SMD:R_0805_2012Metric")
+      (reference "F1") (unit 1) (value "500 mA") (footprint "Resistor_SMD:R_0805_2012Metric")
     )
     (path "/f3b860f9-2f72-404a-8457-15541bcc5c5b"
@@
     )
     (path "/22bd63ac-0dc8-46a4-b634-819479c04be4"
-      (reference "USB1") (unit 1) (value "HRO-TYPE-C-31-M-13") (footprint "42keebs:Molex-216990_GCT-USB45xx_HRO-TYPE-C-31-M-13x-PiMicro")
+      (reference "USB1") (unit 1) (value "HRO-TYPE-C-31-M-13") (footprint "42keebs:TYPE-C-31-M-14-PiMicro")
     )
     (path "/dec5c5bc-8eeb-4827-91ed-4f4f63dc849a"
